Commit message: Change kinematic tree in justina_simple urdf But still unchanged in matlab files

File: catkin_ws/src/hardware/robot_description/justina_simple.urdf (robot description, URDF)
Before this commit: robot justina, 37 links, 36 joints
Links:
- removed link left_arm_link0
- link left_arm_link1: mass None -> 0.35; geometry visual box size=0.07 0.08 0.05
- link left_arm_link2: mass None -> 0.2
- link left_arm_link3: mass None -> 0.18; geometry visual box size=0.075 0.05 0.05
- link left_arm_link4: mass None -> 0.18; geometry visual box size=0.18 0.04 0.04
- link left_arm_link5: mass None -> 0.18; geometry visual box size=0.045 0.05 0.05
- link left_arm_link6: mass None -> 0.15; geometry visual box size=0.1 0.04 0.04
- link left_arm_link7: mass None -> 0.15; geometry visual box size=0.06 0.04 0.04
Joints:
- removed joint la_0_joint
- joint la_1_joint: axis 0 0 1 -> 0 -1 0; limit lower=0 upper=0 effort=0 velocity=0 -> lower=-3.0 upper=3.0 effort=1000 velocity=10; origin xyz=0.055 0.09 0 rpy=1.5708 0 0 -> xyz=0.055 0.09 0 rpy=0 0 0
- joint la_2_joint: axis 0 0 1 -> 0 0 -1; limit lower=0 upper=0 effort=0 velocity=0 -> lower=-3.0 upper=3.0 effort=1000 velocity=10; origin xyz=0.0603 0 0 rpy=1.5708 0 0 -> xyz=0.0603 0 0 rpy=0 0 0
- joint la_3_joint: axis 0 0 1 -> 1 0 0; limit lower=0 upper=0 effort=0 velocity=0 -> lower=-3.0 upper=3.0 effort=1000 velocity=10; origin xyz=0.0 0 0 rpy=1.5708 0 1.5708 -> xyz=0.0 0 0 rpy=0 0 0
- joint la_4_joint: axis 0 0 1 -> 0 -1 0; limit lower=0 upper=0 effort=0 velocity=0 -> lower=-3.0 upper=3.0 effort=1000 velocity=10; origin xyz=0 0 0.27 rpy=-1.5708 0 -1.5708 -> xyz=0.27 0 0 rpy=0 0 0
- joint la_5_joint: axis 0 0 1 -> 1 0 0; limit lower=0 upper=0 effort=0 velocity=0 -> lower=-3.0 upper=3.0 effort=1000 velocity=10; origin xyz=0.0 0 0 rpy=1.5708 0 0 -> xyz=0.0 0 0 rpy=0 0 0
- joint la_6_joint: axis 0 0 1 -> 0 -1 0; limit lower=0 upper=0 effort=0 velocity=0 -> lower=-3.0 upper=3.0 effort=1000 velocity=10; origin xyz=0 0 0.2126 rpy=-1.5708 0 0 -> xyz=0.2126 0 0 rpy=0 0 0
- joint la_7_joint: axis 0 0 1 -> 1 0 0; limit lower=0 upper=0 effort=0 velocity=0 -> lower=-3.0 upper=3.0 effort=1000 velocity=10; origin xyz=0.0 0 0 rpy=1.5708 0 0 -> xyz=0.0 0 0 rpy=0 0 0
- joint la_grip_center_joint: origin xyz=0 0 0.13 rpy=0 0 0 -> xyz=0.13 0 0 rpy=0 0 0
- joint la_grip_left: axis 0 0 1 -> (none); limit lower=0 upper=0 effort=0 velocity=0 -> (none); origin xyz=0 -0.04 0 rpy=0 1.5708 0 -> xyz=0 -0.04 0 rpy=0 0 0
- joint la_grip_right: axis 0 0 1 -> (none); limit lower=0 upper=0 effort=0 velocity=0 -> (none); origin xyz=0 0.04 0 rpy=0 -1.5708 0 -> xyz=0 0.04 0 rpy=0 0 0
