Commit message: Reorder simulink models in subsystems for easier visualization. Add control and smo gaing setting by ros parameters Change masses in simulated models

File: matlab_files/7DOF/JustinaLeftArm.urdf (robot description, URDF)
Before this commit: robot JustinaLeftArm, 11 links, 10 joints
Links:
- link left_arm_link1: mass 0.3 -> 0.35
- link left_arm_link2: mass 0.3 -> 0.2
- link left_arm_link3: mass 0.3 -> 0.18
- link left_arm_link4: mass 0.3 -> 0.18
- link left_arm_link5: mass 0.3 -> 0.18
- link left_arm_link6: mass 0.3 -> 0.15
- link left_arm_link7: mass 0.3 -> 0.15

Commit message: Correct sampling rates of params

File: matlab_files/7DOF/JustinaLeftArm.urdf (robot description, URDF)
Before this commit: robot JustinaLeftArm, 11 links, 10 joints
Joints:
- joint la_1_joint: limit lower=-1.570795 upper=1.570795 effort=1000.0 velocity=0.5 -> lower=-3.0 upper=3.0 effort=1000 velocity=10
- joint la_2_joint: limit lower=-1.570795 upper=1.570795 effort=1000.0 velocity=0.5 -> lower=-3.0 upper=3.0 effort=1000 velocity=10
- joint la_3_joint: limit lower=-1.570795 upper=1.570795 effort=1000.0 velocity=0.5 -> lower=-3.0 upper=3.0 effort=1000 velocity=10
- joint la_4_joint: limit lower=-1.570795 upper=1.570795 effort=1000.0 velocity=0.5 -> lower=-3.0 upper=3.0 effort=1000 velocity=10
- joint la_5_joint: limit lower=-1.570795 upper=1.570795 effort=1000.0 velocity=0.5 -> lower=-3.0 upper=3.0 effort=1000 velocity=10
- joint la_6_joint: limit lower=-1.570795 upper=1.570795 effort=1000.0 velocity=0.5 -> lower=-3.0 upper=3.0 effort=1000 velocity=10
- joint la_7_joint: limit lower=-1.570795 upper=1.570795 effort=1000.0 velocity=0.5 -> lower=-3.0 upper=3.0 effort=1000 velocity=10

Commit message: Change kinematic tree in urdf in matlab files

File: matlab_files/7DOF/JustinaLeftArm.urdf (robot description, URDF)
Before this commit: robot JustinaLeftArm, 11 links, 10 joints
Links:
- link left_arm_link1: geometry visual box size=0.07 0.08 0.05
- link left_arm_link3: geometry visual box size=0.075 0.05 0.05
- link left_arm_link4: geometry visual box size=0.18 0.04 0.04
- link left_arm_link5: geometry visual box size=0.045 0.05 0.05
- link left_arm_link6: geometry visual box size=0.1 0.04 0.04
- link left_arm_link7: geometry visual box size=0.06 0.04 0.04
Joints:
- joint la_1_joint: axis 0 0 1 -> 0 -1 0; origin xyz=0.055 0.09 0 rpy=1.5708 0 0 -> xyz=0.055 0.09 0 rpy=0 0 0
- joint la_2_joint: axis 0 0 1 -> 0 0 -1; origin xyz=0.0603 0 0 rpy=1.5708 0 0 -> xyz=0.0603 0 0 rpy=0 0 0
- joint la_3_joint: axis 0 0 1 -> 1 0 0; origin xyz=0.0 0 0 rpy=1.5708 0 1.5708 -> xyz=0.0 0 0 rpy=0 0 0
- joint la_4_joint: axis 0 0 1 -> 0 -1 0; origin xyz=0 0 0.27 rpy=-1.5708 0 -1.5708 -> xyz=0.27 0 0 rpy=0 0 0
- joint la_5_joint: axis 0 0 1 -> 1 0 0; origin xyz=0.0 0 0 rpy=1.5708 0 0 -> xyz=0.0 0 0 rpy=0 0 0
- joint la_6_joint: axis 0 0 1 -> 0 -1 0; origin xyz=0 0 0.2126 rpy=-1.5708 0 0 -> xyz=0.2126 0 0 rpy=0 0 0
- joint la_7_joint: axis 0 0 1 -> 1 0 0; origin xyz=0.0 0 0 rpy=1.5708 0 0 -> xyz=0.0 0 0 rpy=0 0 0
- joint la_grip_center_joint: origin xyz=0 0 0.13 rpy=0 0 0 -> xyz=0.13 0 0 rpy=0 0 0
- joint la_grip_left: origin xyz=0 -0.04 0 rpy=0 1.5708 0 -> xyz=0 -0.04 0 rpy=0 0 0
- joint la_grip_right: origin xyz=0 0.04 0 rpy=0 -1.5708 0 -> xyz=0 0.04 0 rpy=0 0 0
